File: kicad/portero-bot-v2.kicad_sch (KiCad schematic)
At the start: 77 parts, among them J1 DC005, J2 HR911105A, J3 USB Micro B, J4 KF301-2P, J5 KF301-2P, J6 KF301-2P, J7 Pin Header 01x04 2.54mm Verti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, K1 SRD-05VDC-SL-C, K2 SRD-05VDC-SL-C, K3 SRD-05VDC-SL-C, Q1 2N2222A, Q2 2N2222A, Q3 2N2222A, SW1 KH-6X6X5H-STM, SW2 KH-6X6X5H-STM, U1 ESP32-WROOM-32E-N16, U2 W5500, U3 CH340C, U4 MP2307DN-HW-LF-Z, U5 MP2307DN-HW-LF-Z, Y1 NX3225GA-25MHZ-STD-CRG-2

Commit message: feat(pcb): silkscreen, Edge.Cuts, LEDs corregidos, refs normalizadas
- 13 etiquetas gr_text en F.SilkS (BOOT/RESET/3V3/5V/ENTRADA/SALIDA/PEATONAL)
- Edge.Cuts 117.5x104.5mm via pcbnew SHAPE_T_RECT
- .kicad_dru: drill minimo 0.2mm para vias termicas ESP32
- LEDs: footprint inductor->LED_0603_1608Metric (5 componentes)
- Referencias normalizadas: LED1-5, SW1-2, J4-6, MH1-4 (requerido para freerouting DSN)
- Net "Net 2" renombrada a VIN_FUSED
- DRC: 0 errores reales, 170 unconnected (ruteo pendiente)

Co-Authored-By: Claude Sonnet 4.6 <noreply@anthropic.com>
Parts:
- LED1, LED2, LED3, LED4, LED5: footprint Inductor_SMD:L_6.3x6.3_H3 -> LED_SMD:LED_0603_1608Metric
Connections:
- net Net 2 renamed VIN_FUSED
